File: ir-repeater-booster.kicad_pcb (KiCad board)
At the start: 2 copper layers, 48.8 x 47.2 mm, 35 parts, among them J1 DC_IN, J2 RJ45_LED_Shielded, U1 HT7550-1, U2 ST3485EBDR, U3 HT7533-1

Commit message: Finishing work for 1.0.0 to fabricate
Parts:
- J1: footprint Connector_BarrelJack:BarrelJack_CUI_PJ-102AH_Horizontal -> Connector_BarrelJack:BarrelJack_Wuerth_6941xx301002
- JP3: value DIR -> REDE
Routing:
- net +12V: track 46.7 -> 44.2 mm
- net GND: vias 3 -> 8
Other:
- board text added: "JLCJLCJLCJLC"
- board text added: "idle.to/17"

Commit message: 1.1.0 updates
Parts:
- removed D2, D3: SS14, Diode_SMD:D_SMA
- removed JP3: REDE, Jumper:SolderJumper-2_P1.3mm_Bridged_RoundedPad1.0x1.5mm
- added C5: 10u, Capacitor_SMD:C_1206_3216Metric, F.Cu at (88.1, 71.1)
- added C6: 10u, Capacitor_SMD:C_1206_3216Metric, F.Cu at (83.1, 63.2)
- added TP10: GND, TestPoint:TestPoint_Pad_D2.0mm, F.Cu at (66.5, 60.5)
- added U4: 74HC14, Package_SO:SOIC-14_3.9x8.7mm_P1.27mm, F.Cu at (90.4, 65.8)
- R4: value 270 -> 560; footprint Resistor_SMD:R_0805_2012Metric -> Resistor_SMD:R_0603_1608Metric
- R5: value 270 -> 1k2; footprint Resistor_SMD:R_0805_2012Metric -> Resistor_SMD:R_0603_1608Metric
- moved R3 15.4 mm to (87.6, 79.0)
- moved R1 15.2 mm to (82.5, 67.1)
- moved R4 14.0 mm to (98.0, 82.0)
- moved R2 8.07 mm to (103.4, 80.0)
- moved TP5 7.91 mm to (96.5, 77.0)
- moved TP6 7.91 mm to (96.5, 73.7)
- moved U2 7.91 mm to (89.7, 75.2)
- moved TP1 6.27 mm to (83.3, 73.7)
- moved TP2 6.27 mm to (83.3, 77.0)
- moved TP3 6.27 mm to (83.3, 70.4)
- moved TP4 6.27 mm to (83.3, 80.3)
- moved C3 4.52 mm to (73.4, 78.2)
- moved C4 4.52 mm to (73.4, 70.6)
- moved U3 4.52 mm to (73.4, 74.4)
- moved C1 4.13 mm to (65.8, 78.2)
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Connections:
- J2 pad 1: /A -> /485+
- J2 pad 10: /YLED_A -> /GLED_A
- J2 pad 11: GND -> /YLED_C
- J2 pad 12: /GLED_A -> /YLED_A
- J2 pad 2: /B -> /485-
- J2 pad 9: /YLED_C -> GND
- JP1 pad 1: /B -> /485+
- JP2 pad 2: /!RE -> /DE
- R1 pad 1: +5V -> GND
- R1 pad 2: /TXD -> Net-(R1-Pad2)
- R2 pad 2: /A -> /485-
- R3 pad 1: /!RE -> /DE
- R5 pad 1: +3V3 -> +5V
- RX1 pad 5: /RXD -> /RXOUT
- TP1 pad 1: /!RE -> GND
- TP5 pad 1: /A -> /485+
- TP6 pad 1: /B -> /485-
- TX1 pad 5: /TXD -> Net-(R1-Pad2)
- U2 pad 2: /!RE -> GND
- U2 pad 6: /A -> /485+
- U2 pad 7: /B -> /485-
Routing:
- net GND: track 6.42 -> 57.1 mm
- net +5V: track 50.2 -> 97.5 mm, vias 2 -> 1
- net /A: track 36.7 -> 0.00 mm
- net /485+: track 0.00 -> 34.9 mm
- net /B: track 34.3 -> 0.00 mm, vias 1 -> 0
- net /485-: track 0.00 -> 32.0 mm
- net /!RE: track 31.9 -> 0.00 mm, vias 3 -> 0
- net /DE: track 6.89 -> 36.9 mm, vias 0 -> 2
- net /TXD: track 52.6 -> 23.9 mm, vias 0 -> 2
- net +3V3: track 108.4 -> 81.7 mm, vias 0 -> 3
- net /RXOUT: track 0.00 -> 22.4 mm
- net /RXD: track 31.0 -> 13.1 mm
- net /YLED_C: track 10.8 -> 25.2 mm
- net Net-(R1-Pad2): track 0.00 -> 13.3 mm, vias 0 -> 1
- net /YLED_A: track 10.7 -> 3.05 mm, vias 1 -> 0
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Other:
- board text added: "v1.1.0"
- board text removed: "v1.0.0"
