File: ir-repeater-booster.sch (KiCad schematic (older format))
At the start: 21 parts, among them J1 DC_IN, J2 RJ45_LED_Shielded, U1 HT7550-1, U2 ST3485EBDR, U3 HT7533-1

Commit message: Stashing progress
Parts:
- added H1, H2, H3, H4: MountingHole, MountingHole:MountingHole_3.2mm_M3, symbol Mechanical:MountingHole
- added JP3: REDE, Jumper:SolderJumper-2_P1.3mm_Bridged_RoundedPad1.0x1.5mm, symbol Device:Jumper
- added TP1: !RE, TestPoint:TestPoint_Pad_D2.0mm, symbol Connector:TestPoint
- added TP2: DE, TestPoint:TestPoint_Pad_D2.0mm, symbol Connector:TestPoint
- added TP3: RXD, TestPoint:TestPoint_Pad_D2.0mm, symbol Connector:TestPoint
- added TP4: TXD, TestPoint:TestPoint_Pad_D2.0mm, symbol Connector:TestPoint
- added TP5: A, TestPoint:TestPoint_Pad_D2.0mm, symbol Connector:TestPoint
- added TP6: B, TestPoint:TestPoint_Pad_D2.0mm, symbol Connector:TestPoint
- added TP7: 12V, TestPoint:TestPoint_Pad_D2.0mm, symbol Connector:TestPoint
- added TP8: 5V, TestPoint:TestPoint_Pad_D2.0mm, symbol Connector:TestPoint
- added TP9: 3V3, TestPoint:TestPoint_Pad_D2.0mm, symbol Connector:TestPoint
Connections:
- net labels added: !RE, DE
- net labels removed: DIR
- wire segments 88 -> 99
Other:
- moved on the sheet: JP1, JP2, R2, R3

Commit message: Finishing work for 1.0.0 to fabricate
Parts:
- J1: footprint Connector_BarrelJack:BarrelJack_CUI_PJ-102AH_Horizontal -> Connector_BarrelJack:BarrelJack_Wuerth_6941xx301002
Changed lines of the file:
@@
 F 0 "J1" H 1107 1717 50  0000 C CNN
 F 1 "DC_IN" H 1107 1626 50  0000 C CNN
-F 2 "Connector_BarrelJack:BarrelJack_CUI_PJ-102AH_Horizontal" H 1100 1360 50  0001 C CNN
+F 2 "Connector_BarrelJack:BarrelJack_Wuerth_6941xx301002" H 1100 1360 50  0001 C CNN
 F 3 "~" H 1100 1360 50  0001 C CNN
 	1    1050 1400

Commit message: 1.1.0 updates
Parts:
- removed D2, D3: SS14, Diode_SMD:D_SMA, symbol Device:D_Schottky
- removed JP3: REDE, Jumper:SolderJumper-2_P1.3mm_Bridged_RoundedPad1.0x1.5mm, symbol Device:Jumper
- added C5, C6: 10u, Capacitor_SMD:C_1206_3216Metric, symbol Device:C
- added TP10: GND, TestPoint:TestPoint_Pad_D2.0mm, symbol Connector:TestPoint
- added U4: 74HC14, Package_SO:SOIC-14_3.9x8.7mm_P1.27mm, symbol 74xx:74HC14
- R4: value 270 -> 560; footprint Resistor_SMD:R_0805_2012Metric -> Resistor_SMD:R_0603_1608Metric; Description 270Ω ±1% 0.125W ±100ppm/℃ 0805 Chip Resistor - Surface Moun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 -> 560Ω ±1% 0.1W ±100ppm/℃ 0603 Chip Resistor - Surface Mount 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; JEDEC Package Name 0805 -> 0603; Manufacturer Part Number 0805W8F2700T5E -> 0603WAF5600T5E; Package Comments (none) -> Imperial; Vendor 1 Link https://lcsc.com/product-detail/Chip-Resistor-Surface-Mount_Uniroyal-Elec-0805W8F2700T5E_C17590.html/?href=jlc-SMT -> https://lcsc.com/product-detail/Chip-Resistor-Surface-Mount_Uniroyal-Elec-0603WAF5600T5E_C23204.html/?href=jlc-SMT; Vendor 1 Part Number C17590 -> C23204; Vendor 1 Price @1 $0.0027 -> $0.0021; Vendor 1 Pricing Date 2021-03-03 -> 2021-03-20
- R5: value 270 -> 1k2; footprint Resistor_SMD:R_0805_2012Metric -> Resistor_SMD:R_0603_1608Metric; Description 270Ω ±1% 0.125W ±100ppm/℃ 0805 Chip Resistor - Surface Moun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 -> 1.2kΩ ±1% 0.1W ±100ppm/℃ 0603 Chip Resistor - Surface Mount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; JEDEC Package Name 0805 -> 0603; Manufacturer Part Number 0805W8F2700T5E -> 0603WAF1201T5E; Package Comments (none) -> Imperial; Vendor 1 Link https://lcsc.com/product-detail/Chip-Resistor-Surface-Mount_Uniroyal-Elec-0805W8F2700T5E_C17590.html/?href=jlc-SMT -> https://lcsc.com/product-detail/Chip-Resistor-Surface-Mount_Uniroyal-Elec-0603WAF1201T5E_C22765.html/?href=jlc-SMT; Vendor 1 Part Number C17590 -> C22765; Vendor 1 Price @1 $0.0027 -> $0.0019; Vendor 1 Pricing Date 2021-03-03 -> 2021-03-20
Connections:
- net labels added: 485+, 485-, RXOUT
- wire segments 99 -> 107
Other:
- note added: "Hex inverter used to square and shift I/O to 5V"
- moved on the sheet: D1, J1, J2, JP1, JP2, R1, R2, R3, RX1, TP1, TP2, TP3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
